Commit message: commit

File: models/physics.urdf (robot description, URDF)
Before this commit: robot dumpUrdf, 95 links, 94 joints
Joints:
- joint left_hip_rz: origin xyz=0 0 0 rpy=0 0 0 -> xyz=0 0 0 rpy=0.05 0 0
- joint left_shoulder_rz: origin xyz=0 0 0 rpy=0 0 0 -> xyz=0 0 0 rpy=-0.7 0 0
- joint right_hip_rz: origin xyz=0 0 0 rpy=0 0 0 -> xyz=0 0 0 rpy=-0.05 0 0
- joint right_shoulder_rz: origin xyz=0 0 0 rpy=0 0 0 -> xyz=0 0 0 rpy=0.7 0 0

Commit message: 添加debug代码

File: models/physics.urdf (robot description, URDF)
Before this commit: robot dumpUrdf, 95 links, 94 joints
Joints:
- joint left_shoulder_rz: origin xyz=0 0 0 rpy=-0.7 0 0 -> xyz=0 0 0 rpy=0 0 0
- joint right_shoulder_rz: origin xyz=0 0 0 rpy=0.7 0 0 -> xyz=0 0 0 rpy=0 0 0

Commit message: 添加urdf修改

File: models/physics.urdf (robot description, URDF)
Before this commit: robot dumpUrdf, 95 links, 94 joints
Joints:
- joint right_clavicle_rx: origin xyz=-0.02371300000000001 -0.08099875 0.1105722 rpy=0 0 0 -> xyz=-0.02371300000000001 -0.08099875 0.1105722 rpy=0 3.14 0

Commit message: Update physics.urdf

File: models/physics.urdf (robot description, URDF)
Before this commit: robot dumpUrdf, 95 links, 94 joints
Joints:
- joint right_clavicle_rx: origin xyz=-0.02371300000000001 -0.08099875 0.1105722 rpy=0 3.14 0 -> xyz=-0.02371300000000001 -0.08099875 0.1105722 rpy=0 0 0
